Commit message: update the vehicle_simulation models

File: src/vehicle_simulation/gazebo/sd_twizy_model/streetdrone_model/sd_description/urdf/bases/sd_twizy_body.gazebo.xacro (robot description, xacro)
@@ -1,5 +1,5 @@
 <?xml version="1.0"?>
 <!--
-Copyright (c) 2020 StreetDrone Limited
+Copyright (c) 2019 StreetDrone Limited
 Author:  Efimia Panagiotaki
 All rights reserved

File: src/vehicle_simulation/gazebo/sd_twizy_model/streetdrone_model/sd_description/urdf/bases/sd_twizy_body.urdf.xacro (robot description, xacro)
@@ -1,5 +1,5 @@
 <?xml version="1.0"?>
 <!--
-Copyright (c) 2020 StreetDrone Limited
+Copyright (c) 2019 StreetDrone Limited
 Author:  Efimia Panagiotaki
 All rights reserved

File: src/vehicle_simulation/gazebo/sd_twizy_model/streetdrone_model/sd_description/urdf/sd_twizy.urdf.xacro (robot description, xacro)
@@ -1,5 +1,5 @@
 <?xml version="1.0"?>
 <!--
-Copyright (c) 2020 StreetDrone Limited
+Copyright (c) 2019 StreetDrone Limited
 Author:  Efimia Panagiotaki
 All rights reserved
@@ -25,28 +25,28 @@
     <origin xyz="-0.681 0 1.445" rpy="0 -${1.5*M_PI/180.0} 0"/>
   </xacro:VLP-16>
-  <xacro:blackfly_camera frlr_prefix="front" lrc_prefix="left">
+  <xacro:sekonix_camera frlr_prefix="front" lrc_prefix="left">
     <origin xyz="-0.04 0.12 1.3" rpy="0 0.087 0"/>
-  </xacro:blackfly_camera>
-  <xacro:blackfly_camera frlr_prefix="front" lrc_prefix="right">
+  </xacro:sekonix_camera>
+  <xacro:sekonix_camera frlr_prefix="front" lrc_prefix="right">
     <origin xyz="-0.04 -0.12 1.3" rpy="0 0.087 0"/>
-  </xacro:blackfly_camera>
-  <xacro:blackfly_camera frlr_prefix="front" lrc_prefix="center">
+  </xacro:sekonix_camera>
+  <xacro:sekonix_camera frlr_prefix="front" lrc_prefix="center">
     <origin xyz="-0.04 0 1.3" rpy="0 0.087 0"/>
-  </xacro:blackfly_camera>
-  <xacro:blackfly_camera frlr_prefix="rear" lrc_prefix="center">
+  </xacro:sekonix_camera>
+  <xacro:sekonix_camera frlr_prefix="rear" lrc_prefix="center">
     <origin xyz="-1.26 0 1.28" rpy="0 0.2618 3.14"/>
-  </xacro:blackfly_camera>
-  <xacro:blackfly_camera frlr_prefix="right" lrc_prefix="forward">
+  </xacro:sekonix_camera>
+  <xacro:sekonix_camera frlr_prefix="right" lrc_prefix="forward">
     <origin xyz="-0.95 -0.42 1.2" rpy="0 0.244 -1.12"/>
-  </xacro:blackfly_camera>
-  <xacro:blackfly_camera frlr_prefix="right" lrc_prefix="rearward">
+  </xacro:sekonix_camera>
+  <xacro:sekonix_camera frlr_prefix="right" lrc_prefix="rearward">
     <origin xyz="-1.05 -0.42 1.2" rpy="0 0.244 -2.18"/>
-  </xacro:blackfly_camera>
-  <xacro:blackfly_camera frlr_prefix="left" lrc_prefix="forward">
+  </xacro:sekonix_camera>
+  <xacro:sekonix_camera frlr_prefix="left" lrc_prefix="forward">
     <origin xyz="-0.95 0.4 1.2" rpy="0 0.2967 1.12"/>
-  </xacro:blackfly_camera>
-  <xacro:blackfly_camera frlr_prefix="left" lrc_prefix="rearward">
+  </xacro:sekonix_camera>
+  <xacro:sekonix_camera frlr_prefix="left" lrc_prefix="rearward">
     <origin xyz="-1.05 0.39 1.2" rpy="0 0.2967 2.18"/>
-  </xacro:blackfly_camera>
+  </xacro:sekonix_camera>
   <gazebo>
     <plugin name="sd_control" filename="libSdControlPlugin.so">

File: src/vehicle_simulation/gazebo/sd_twizy_model/streetdrone_model/sd_description/urdf/sensors/cameras.urdf.xacro (robot description, xacro)
@@ -1,10 +1,10 @@
 <?xml version="1.0"?>
 <!--
-Copyright (c) 2020 StreetDrone Limited
+Copyright (c) 2019 StreetDrone Limited
 Author:  Efimia Panagiotaki
 All rights reserved
 -->
-<robot xmlns:xacro="http://www.ros.org/wiki/xacro" name="blackfly_camera">
-    <xacro:macro name="blackfly_camera" params="frlr_prefix lrc_prefix *origin">
+<robot xmlns:xacro="http://www.ros.org/wiki/xacro" name="sekonix_camera">
+  <xacro:macro name="sekonix_camera" params="frlr_prefix lrc_prefix *origin">
     <joint name="${frlr_prefix}_${lrc_prefix}_camera_joint" type="fixed">
       <axis xyz="0 1 0" />
@@ -44,53 +44,53 @@
     </joint>
     <link name="${frlr_prefix}_${lrc_prefix}_camera_link_optical"/>
-        <gazebo reference="${frlr_prefix}_${lrc_prefix}_camera_link">
-            <mu1>0.2</mu1>
-            <mu2>0.2</mu2>
-            <material>Gazebo/Red</material>
-            <sensor type="camera" name="${frlr_prefix}_${lrc_prefix}_camera">
-                <update_rate>30.0</update_rate>
-                <camera name="head">
-                    <horizontal_fov>2.09</horizontal_fov>
-                    <image>
-                        <width>1920</width>
-                        <height>1200</height>
-                        <format>R8G8B8</format>
-                    </image>
-                    <clip>
-                        <near>0.1</near>
-                        <far>30</far>
-                    </clip>
-                    <noise>
-                        <type>gaussian</type>
-                        <!-- Noise is sampled independently per pixel on each frame.
-                             That pixel's noise value is added to each of its color
-                             channels, which at that point lie in the range [0,1]. -->
-                        <mean>0.0</mean>
-                        <stddev>0.007</stddev>
-                    </noise>
-                </camera>
-                <plugin name="${frlr_prefix}_${lrc_prefix}_camera_controller" filename="libgazebo_ros_camera.so">
-                    <alwaysOn>true</alwaysOn>
-                    <updateRate>0.0</updateRate>
-                    <cameraName>sd_twizy/${frlr_prefix}_${lrc_prefix}_camera</cameraName>
-                    <imageTopicName>image_raw</imageTopicName>
-                    <cameraInfoTopicName>camera_info</cameraInfoTopicName>
-                    <frameName>${frlr_prefix}_${lrc_prefix}_camera_link_optical</frameName>
-                    <!-- setting hackBaseline to anything but 0.0 will cause a misalignment
-                        between the gazebo sensor image and the frame it is supposed to
-                        be attached to -->
-                    <hackBaseline>0.0</hackBaseline>
-                    <distortionK1>0.0</distortionK1>
-                    <distortionK2>0.0</distortionK2>
-                    <distortionK3>0.0</distortionK3>
-                    <distortionT1>0.0</distortionT1>
-                    <distortionT2>0.0</distortionT2>
-                    <CxPrime>0</CxPrime>
-                    <Cx>0.0</Cx>
-                    <Cy>0.0</Cy>
-                    <focalLength>0.0</focalLength>
-                </plugin>
-            </sensor>
-        </gazebo>
+    <gazebo reference="${frlr_prefix}_${lrc_prefix}_camera_link">
+      <mu1>0.2</mu1>
+      <mu2>0.2</mu2>
+      <material>Gazebo/Red</material>
+      <sensor type="camera" name="${frlr_prefix}_${lrc_prefix}_camera">
+        <update_rate>30.0</update_rate>
+        <camera name="head">
+          <horizontal_fov>2.09</horizontal_fov>
+          <image>
+            <width>1928</width>
+            <height>1208</height>
+            <format>R8G8B8</format>
+          </image>
+          <clip>
+            <near>0.1</near>
+            <far>30</far>
+          </clip>
+          <noise>
+            <type>gaussian</type>
+            <!-- Noise is sampled independently per pixel on each frame.
+                 That pixel's noise value is added to each of its color
+                 channels, which at that point lie in the range [0,1]. -->
+            <mean>0.0</mean>
+            <stddev>0.007</stddev>
+          </noise>
+        </camera>
+        <plugin name="${frlr_prefix}_${lrc_prefix}_camera_controller" filename="libgazebo_ros_camera.so">
+          <alwaysOn>true</alwaysOn>
+          <updateRate>0.0</updateRate>
+          <cameraName>sd_twizy/${frlr_prefix}_${lrc_prefix}_camera</cameraName>
+          <imageTopicName>image_raw</imageTopicName>
+          <cameraInfoTopicName>camera_info</cameraInfoTopicName>
+          <frameName>${frlr_prefix}_${lrc_prefix}_camera_link_optical</frameName>
+          <!-- setting hackBaseline to anything but 0.0 will cause a misalignment
+               between the gazebo sensor image and the frame it is supposed to
+               be attached to -->
+          <hackBaseline>0.0</hackBaseline>
+          <distortionK1>0.0</distortionK1>
+          <distortionK2>0.0</distortionK2>
+          <distortionK3>0.0</distortionK3>
+          <distortionT1>0.0</distortionT1>
+          <distortionT2>0.0</distortionT2>
+          <CxPrime>0</CxPrime>
+          <Cx>0.0</Cx>
+          <Cy>0.0</Cy>
+          <focalLength>0.0</focalLength>
+        </plugin>
+      </sensor>
+    </gazebo>
   </xacro:macro>
 </robot>

File: src/vehicle_simulation/gazebo/sd_twizy_model/streetdrone_model/sd_description/urdf/wheels/sd_twizy_suspension.urdf.xacro (robot description, xacro)
@@ -1,5 +1,5 @@
 <?xml version="1.0"?>
 <!--
-Copyright (c) 2020 StreetDrone Limited
+Copyright (c) 2019 StreetDrone Limited
 Author:  Efimia Panagiotaki
 All rights reserved

Commit message: Bring branch up-to-date

File: src/vehicle_simulation/gazebo/sd_twizy_model/streetdrone_model/sd_description/urdf/bases/sd_twizy_body.gazebo.xacro (robot description, xacro)
@@ -1,5 +1,5 @@
 <?xml version="1.0"?>
 <!--
-Copyright (c) 2019 StreetDrone Limited
+Copyright (c) 2020 StreetDrone Limited
 Author:  Efimia Panagiotaki
 All rights reserved

File: src/vehicle_simulation/gazebo/sd_twizy_model/streetdrone_model/sd_description/urdf/bases/sd_twizy_body.urdf.xacro (robot description, xacro)
@@ -1,5 +1,5 @@
 <?xml version="1.0"?>
 <!--
-Copyright (c) 2019 StreetDrone Limited
+Copyright (c) 2020 StreetDrone Limited
 Author:  Efimia Panagiotaki
 All rights reserved

File: src/vehicle_simulation/gazebo/sd_twizy_model/streetdrone_model/sd_description/urdf/sd_twizy.urdf.xacro (robot description, xacro)
@@ -1,5 +1,5 @@
 <?xml version="1.0"?>
 <!--
-Copyright (c) 2019 StreetDrone Limited
+Copyright (c) 2020 StreetDrone Limited
 Author:  Efimia Panagiotaki
 All rights reserved
@@ -25,28 +25,28 @@
     <origin xyz="-0.681 0 1.445" rpy="0 -${1.5*M_PI/180.0} 0"/>
   </xacro:VLP-16>
-  <xacro:sekonix_camera frlr_prefix="front" lrc_prefix="left">
+  <xacro:blackfly_camera frlr_prefix="front" lrc_prefix="left">
     <origin xyz="-0.04 0.12 1.3" rpy="0 0.087 0"/>
-  </xacro:sekonix_camera>
-  <xacro:sekonix_camera frlr_prefix="front" lrc_prefix="right">
+  </xacro:blackfly_camera>
+  <xacro:blackfly_camera frlr_prefix="front" lrc_prefix="right">
     <origin xyz="-0.04 -0.12 1.3" rpy="0 0.087 0"/>
-  </xacro:sekonix_camera>
-  <xacro:sekonix_camera frlr_prefix="front" lrc_prefix="center">
+  </xacro:blackfly_camera>
+  <xacro:blackfly_camera frlr_prefix="front" lrc_prefix="center">
     <origin xyz="-0.04 0 1.3" rpy="0 0.087 0"/>
-  </xacro:sekonix_camera>
-  <xacro:sekonix_camera frlr_prefix="rear" lrc_prefix="center">
+  </xacro:blackfly_camera>
+  <xacro:blackfly_camera frlr_prefix="rear" lrc_prefix="center">
     <origin xyz="-1.26 0 1.28" rpy="0 0.2618 3.14"/>
-  </xacro:sekonix_camera>
-  <xacro:sekonix_camera frlr_prefix="right" lrc_prefix="forward">
+  </xacro:blackfly_camera>
+  <xacro:blackfly_camera frlr_prefix="right" lrc_prefix="forward">
     <origin xyz="-0.95 -0.42 1.2" rpy="0 0.244 -1.12"/>
-  </xacro:sekonix_camera>
-  <xacro:sekonix_camera frlr_prefix="right" lrc_prefix="rearward">
+  </xacro:blackfly_camera>
+  <xacro:blackfly_camera frlr_prefix="right" lrc_prefix="rearward">
     <origin xyz="-1.05 -0.42 1.2" rpy="0 0.244 -2.18"/>
-  </xacro:sekonix_camera>
-  <xacro:sekonix_camera frlr_prefix="left" lrc_prefix="forward">
+  </xacro:blackfly_camera>
+  <xacro:blackfly_camera frlr_prefix="left" lrc_prefix="forward">
     <origin xyz="-0.95 0.4 1.2" rpy="0 0.2967 1.12"/>
-  </xacro:sekonix_camera>
-  <xacro:sekonix_camera frlr_prefix="left" lrc_prefix="rearward">
+  </xacro:blackfly_camera>
+  <xacro:blackfly_camera frlr_prefix="left" lrc_prefix="rearward">
     <origin xyz="-1.05 0.39 1.2" rpy="0 0.2967 2.18"/>
-  </xacro:sekonix_camera>
+  </xacro:blackfly_camera>
   <gazebo>
     <plugin name="sd_control" filename="libSdControlPlugin.so">

File: src/vehicle_simulation/gazebo/sd_twizy_model/streetdrone_model/sd_description/urdf/sensors/cameras.urdf.xacro (robot description, xacro)
@@ -1,10 +1,10 @@
 <?xml version="1.0"?>
 <!--
-Copyright (c) 2019 StreetDrone Limited
+Copyright (c) 2020 StreetDrone Limited
 Author:  Efimia Panagiotaki
 All rights reserved
 -->
-<robot xmlns:xacro="http://www.ros.org/wiki/xacro" name="sekonix_camera">
-  <xacro:macro name="sekonix_camera" params="frlr_prefix lrc_prefix *origin">
+<robot xmlns:xacro="http://www.ros.org/wiki/xacro" name="blackfly_camera">
+    <xacro:macro name="blackfly_camera" params="frlr_prefix lrc_prefix *origin">
     <joint name="${frlr_prefix}_${lrc_prefix}_camera_joint" type="fixed">
       <axis xyz="0 1 0" />
@@ -44,53 +44,53 @@
     </joint>
     <link name="${frlr_prefix}_${lrc_prefix}_camera_link_optical"/>
-    <gazebo reference="${frlr_prefix}_${lrc_prefix}_camera_link">
-      <mu1>0.2</mu1>
-      <mu2>0.2</mu2>
-      <material>Gazebo/Red</material>
-      <sensor type="camera" name="${frlr_prefix}_${lrc_prefix}_camera">
-        <update_rate>30.0</update_rate>
-        <camera name="head">
-          <horizontal_fov>2.09</horizontal_fov>
-          <image>
-            <width>1928</width>
-            <height>1208</height>
-            <format>R8G8B8</format>
-          </image>
-          <clip>
-            <near>0.1</near>
-            <far>30</far>
-          </clip>
-          <noise>
-            <type>gaussian</type>
-            <!-- Noise is sampled independently per pixel on each frame.
-                 That pixel's noise value is added to each of its color
-                 channels, which at that point lie in the range [0,1]. -->
-            <mean>0.0</mean>
-            <stddev>0.007</stddev>
-          </noise>
-        </camera>
-        <plugin name="${frlr_prefix}_${lrc_prefix}_camera_controller" filename="libgazebo_ros_camera.so">
-          <alwaysOn>true</alwaysOn>
-          <updateRate>0.0</updateRate>
-          <cameraName>sd_twizy/${frlr_prefix}_${lrc_prefix}_camera</cameraName>
-          <imageTopicName>image_raw</imageTopicName>
-          <cameraInfoTopicName>camera_info</cameraInfoTopicName>
-          <frameName>${frlr_prefix}_${lrc_prefix}_camera_link_optical</frameName>
-          <!-- setting hackBaseline to anything but 0.0 will cause a misalignment
-               between the gazebo sensor image and the frame it is supposed to
-               be attached to -->
-          <hackBaseline>0.0</hackBaseline>
-          <distortionK1>0.0</distortionK1>
-          <distortionK2>0.0</distortionK2>
-          <distortionK3>0.0</distortionK3>
-          <distortionT1>0.0</distortionT1>
-          <distortionT2>0.0</distortionT2>
-          <CxPrime>0</CxPrime>
-          <Cx>0.0</Cx>
-          <Cy>0.0</Cy>
-          <focalLength>0.0</focalLength>
-        </plugin>
-      </sensor>
-    </gazebo>
+        <gazebo reference="${frlr_prefix}_${lrc_prefix}_camera_link">
+            <mu1>0.2</mu1>
+            <mu2>0.2</mu2>
+            <material>Gazebo/Red</material>
+            <sensor type="camera" name="${frlr_prefix}_${lrc_prefix}_camera">
+                <update_rate>30.0</update_rate>
+                <camera name="head">
+                    <horizontal_fov>2.09</horizontal_fov>
+                    <image>
+                        <width>1920</width>
+                        <height>1200</height>
+                        <format>R8G8B8</format>
+                    </image>
+                    <clip>
+                        <near>0.1</near>
+                        <far>30</far>
+                    </clip>
+                    <noise>
+                        <type>gaussian</type>
+                        <!-- Noise is sampled independently per pixel on each frame.
+                             That pixel's noise value is added to each of its color
+                             channels, which at that point lie in the range [0,1]. -->
+                        <mean>0.0</mean>
+                        <stddev>0.007</stddev>
+                    </noise>
+                </camera>
+                <plugin name="${frlr_prefix}_${lrc_prefix}_camera_controller" filename="libgazebo_ros_camera.so">
+                    <alwaysOn>true</alwaysOn>
+                    <updateRate>0.0</updateRate>
+                    <cameraName>sd_twizy/${frlr_prefix}_${lrc_prefix}_camera</cameraName>
+                    <imageTopicName>image_raw</imageTopicName>
+                    <cameraInfoTopicName>camera_info</cameraInfoTopicName>
+                    <frameName>${frlr_prefix}_${lrc_prefix}_camera_link_optical</frameName>
+                    <!-- setting hackBaseline to anything but 0.0 will cause a misalignment
+                        between the gazebo sensor image and the frame it is supposed to
+                        be attached to -->
+                    <hackBaseline>0.0</hackBaseline>
+                    <distortionK1>0.0</distortionK1>
+                    <distortionK2>0.0</distortionK2>
+                    <distortionK3>0.0</distortionK3>
+                    <distortionT1>0.0</distortionT1>
+                    <distortionT2>0.0</distortionT2>
+                    <CxPrime>0</CxPrime>
+                    <Cx>0.0</Cx>
+                    <Cy>0.0</Cy>
+                    <focalLength>0.0</focalLength>
+                </plugin>
+            </sensor>
+        </gazebo>
   </xacro:macro>
 </robot>

File: src/vehicle_simulation/gazebo/sd_twizy_model/streetdrone_model/sd_description/urdf/wheels/sd_twizy_suspension.urdf.xacro (robot description, xacro)
@@ -1,5 +1,5 @@
 <?xml version="1.0"?>
 <!--
-Copyright (c) 2019 StreetDrone Limited
+Copyright (c) 2020 StreetDrone Limited
 Author:  Efimia Panagiotaki
 All rights reserved
